File: SmoothieDriver-DC3.brd (EAGLE design)
At the start: 50.8 x 83.8 mm, 89 parts, among them Q2 25mA, Q3 25mA, U1 LPC1114FBD48, U2 MCP4725A0, U3 MCP4725A0, U4 MCP4725A1, U5 MCP1252-33X40I/MS, X1 DRIVER_0, X2 DRIVER_1, X3 DRIVER_2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

Commit message: Prototype 2 as sent to board house
Other:
- board size 50.8 x 83.8 mm -> 50.4 x 83.8 mm
- board text added: "!EN!"
- board text added: "A"
- board text added: "B"
- board text added: "DIR"
- board text added: "Encoder"
- board text added: "Gmot"
- board text added: "Gnd"
- board text added: "Max"
- board text added: "Min"
- board text added: "S"
- board text added: "STEP"
- board text added: "Vcc"
- board text added: "Vmot"
- board text added: "Vout"
- board text added: "http://reprap.org/wiki/IRC"
- board text added: "http://smoothieware.org/"
- board text added: "http://trinitylabs.com/"
- board text removed: "http://www.smoothieware.org/"
- board text removed: "http://www.trinitylabs.com/"
