File: SmoothieDriver-DC3.sch (EAGLE design)
At the start: 89 parts, among them Q2 25mA, Q3 25mA, U1 LPC1114FBD48, U2 MCP4725A0, U3 MCP4725A0, U4 MCP4725A1, U5 MCP1252-33X40I/MS, X1 DRIVER_0, X2 DRIVER_1, X3 DRIVER_2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

Commit message: Prototype 2 as sent to board house
Changed lines of the file:
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@@
 <wire x1="314.96" y1="190.5" x2="314.96" y2="187.96" width="0.1524" layer="91"/>
 <wire x1="314.96" y1="187.96" x2="312.42" y2="187.96" width="0.1524" layer="91"/>
+<label x="317.5" y="185.42" size="1.778" layer="95"/>
 </segment>
 <segment>
@@
 <wire x1="312.42" y1="137.16" x2="314.96" y2="137.16" width="0.1524" layer="91"/>
 <pinref part="U$24" gate="G$1" pin="P$2"/>
+<label x="317.5" y="134.62" size="1.778" layer="95"/>
 </segment>
 <segment>
@@
 <wire x1="312.42" y1="86.36" x2="314.96" y2="86.36" width="0.1524" layer="91"/>
 <pinref part="U$25" gate="G$1" pin="P$2"/>
+<label x="317.5" y="83.82" size="1.778" layer="95"/>
 </segment>
 <segment>
